Commit message: add leapmotino dexpilot retarget

File: holodex/robot/hand/leap/assets/leap_hand_right.urdf (robot description, URDF)
Before this commit: robot leap_right, 28 links, 27 joints
Links:
- removed link dip_retarget
- removed link fingertip_retarget
Joints:
- removed joint dip_retarget_joint
- removed joint fingertip_retarget_joint

Commit message: new mesh

File: holodex/robot/hand/leap/assets/leap_hand_right.urdf (robot description, URDF)
Before this commit: robot leap_right, 26 links, 25 joints
Links:
- link fingertip: geometry collision mesh filename=meshes/visual/fingertip_paxini_fu.obj; visual mesh filename=meshes/visual/fingertip_paxini_fu.obj
- link fingertip_2: geometry collision mesh filename=meshes/visual/fingertip_paxini_fu.obj; visual mesh filename=meshes/visual/fingertip_paxini_fu.obj
- link fingertip_3: geometry collision mesh filename=meshes/visual/fingertip_paxini_fu.obj; visual mesh filename=meshes/visual/fingertip_paxini_fu.obj
- link thumb_fingertip: geometry collision mesh filename=meshes/visual/thumb_fingertip_paxini_fu.obj; visual mesh filename=meshes/visual/thumb_fingertip_paxini_fu.obj

Commit message: new hand urdf

File: holodex/robot/hand/leap/assets/leap_hand_right.urdf (robot description, URDF)
Before this commit: robot leap_right, 26 links, 25 joints
Links:
- added link index_dip_head
- added link middle_dip_head
- added link ring_dip_head
- added link thumb_dip_head
- link dip: geometry collision box size=0.014 0.02 0.004; collision box size=0.014 0.02 0.004
- link dip_2: geometry collision box size=0.014 0.02 0.004; collision box size=0.014 0.02 0.004
- link dip_3: geometry collision box size=0.014 0.02 0.004; collision box size=0.014 0.02 0.004
- link fingertip: geometry collision mesh filename=meshes/visual/fingertip_new_convex.obj; visual mesh filename=meshes/visual/fingertip_new_convex.obj
- link fingertip_2: geometry collision mesh filename=meshes/visual/fingertip_new_convex.obj; visual mesh filename=meshes/visual/fingertip_new_convex.obj
- link fingertip_3: geometry collision mesh filename=meshes/visual/fingertip_new_convex.obj; visual mesh filename=meshes/visual/fingertip_new_convex.obj
- link thumb_fingertip: geometry collision mesh filename=meshes/visual/thumb_fingertip_paxini_convex.obj; visual mesh filename=meshes/visual/thumb_fingertip_paxini_convex.obj
Joints:
- added joint index_dip_retarget: type fixed, parent fingertip, child index_dip_head, origin xyz=0.0 0.0 0.014 rpy=0 0 0
- added joint middle_dip_retarget: type fixed, parent fingertip_2, child middle_dip_head, origin xyz=0.0 0.0 0.014 rpy=0 0 0
- added joint ring_dip_retarget: type fixed, parent fingertip_3, child ring_dip_head, origin xyz=0.0 0.0 0.014 rpy=0 0 0
- added joint thumb_dip_retarget: type fixed, parent thumb_fingertip, child thumb_dip_head, origin xyz=0.0 0.0 -0.014 rpy=0 0 0
- joint base_joint: origin xyz=-0.015 0.038 0.098 rpy=0 -1.57079 0 -> xyz=-0.015 0.038 0.058 rpy=0 -1.57079 0
- joint index_tip: origin xyz=0 -0.036 0.015 rpy=0 0 0 -> xyz=-0.011 -0.029 0.015 rpy=0 0 0
- joint middle_tip: origin xyz=0 -0.036 0.015 rpy=0 0 0 -> xyz=-0.011 -0.029 0.015 rpy=0 0 0
- joint ring_tip: origin xyz=0 -0.036 0.015 rpy=0 0 0 -> xyz=-0.011 -0.029 0.015 rpy=0 0 0
- joint thumb_tip: origin xyz=0 -0.048 -0.015 rpy=0 0 0 -> xyz=-0.011 -0.043 -0.015 rpy=0 0 0

Commit message: Initial commit

File: holodex/robot/hand/leap/assets/leap_hand_right.urdf (robot description, URDF)
Before this commit: robot leap_right, 30 links, 29 joints
Joints:
- joint 10: limit lower=-0.506 upper=1.885 effort=0.95 velocity=8.48 -> lower=-0.506 upper=1.3 effort=0.95 velocity=8.48
- joint 2: limit lower=-0.506 upper=1.885 effort=0.95 velocity=8.48 -> lower=-0.506 upper=1.3 effort=0.95 velocity=8.48
- joint 6: limit lower=-0.506 upper=1.885 effort=0.95 velocity=8.48 -> lower=-0.506 upper=1.3 effort=0.95 velocity=8.48

Commit message: recover original

File: holodex/robot/hand/leap/assets/leap_hand_right.urdf (robot description, URDF)
Before this commit: robot leap_right, 30 links, 29 joints
Joints:
- joint 10: limit lower=-0.506 upper=1.3 effort=0.95 velocity=8.48 -> lower=-0.506 upper=1.885 effort=0.95 velocity=8.48
- joint 2: limit lower=-0.506 upper=1.3 effort=0.95 velocity=8.48 -> lower=-0.506 upper=1.885 effort=0.95 velocity=8.48
- joint 6: limit lower=-0.506 upper=1.3 effort=0.95 velocity=8.48 -> lower=-0.506 upper=1.885 effort=0.95 velocity=8.48

Commit message: fix urdf error

File: holodex/robot/hand/leap/assets/leap_hand_right.urdf (robot description, URDF)
Before this commit: robot leap_right, 30 links, 29 joints
Joints:
- joint 11: origin xyz=0 -0.03609 0.0002 rpy=0 0 0 -> xyz=0 -0.04609 0.0002 rpy=0 0 0
- joint 3: origin xyz=0 -0.0361 0.0002 rpy=0 0 0 -> xyz=0 -0.0461 0.0002 rpy=0 0 0
- joint 7: origin xyz=0 -0.0361 0.0002 rpy=0 0 0 -> xyz=0 -0.0461 0.0002 rpy=0 0 0

Commit message: update Dec version

File: holodex/robot/hand/leap/assets/leap_hand_right.urdf (robot description, URDF)
Before this commit: robot leap_right, 30 links, 29 joints
Joints:
- joint 10: limit lower=-0.506 upper=1.885 effort=0.95 velocity=8.48 -> lower=-0.506 upper=1.3 effort=0.95 velocity=8.48
- joint 11: limit lower=-0.366 upper=2.042 effort=0.95 velocity=8.48 -> lower=-0.366 upper=1.0 effort=0.95 velocity=8.48
- joint 2: limit lower=-0.506 upper=1.885 effort=0.95 velocity=8.48 -> lower=-0.506 upper=1.3 effort=0.95 velocity=8.48
- joint 3: limit lower=-0.366 upper=2.042 effort=0.95 velocity=8.48 -> lower=-0.366 upper=1.0 effort=0.95 velocity=8.48
- joint 6: limit lower=-0.506 upper=1.885 effort=0.95 velocity=8.48 -> lower=-0.506 upper=1.3 effort=0.95 velocity=8.48
- joint 7: limit lower=-0.366 upper=2.042 effort=0.95 velocity=8.48 -> lower=-0.366 upper=1.0 effort=0.95 velocity=8.48
- joint index_tip: origin xyz=-0.011 -0.029 0.015 rpy=0 0 0 -> xyz=-0.001 -0.019 0.015 rpy=0 0 0
- joint middle_tip: origin xyz=-0.011 -0.029 0.015 rpy=0 0 0 -> xyz=-0.011 -0.019 0.015 rpy=0 0 0
- joint ring_tip: origin xyz=-0.011 -0.029 0.015 rpy=0 0 0 -> xyz=-0.011 -0.019 0.015 rpy=0 0 0
- joint thumb_tip: origin xyz=-0.011 -0.043 -0.015 rpy=0 0 0 -> xyz=-0.011 -0.033 -0.015 rpy=0 0 0
